Commit message: modif for online and changing PC

File: src/vacuum/urdf/vacuum.urdf (robot description, URDF)
Before this commit: robot vacuum, 2 links, 1 joints
Links:
- link vacuum_base_link: geometry collision mesh filename=package://vacuum/meshes/tool.STL scale=0.0015 0.0015 0.0015; visual mesh filename=package://vacuum/meshes/tool.STL scale=0.001 0.001 0.001
- link vacuum_tcp: geometry collision cylinder length=0.15 radius=0.03; visual cylinder length=0.15 radius=0.015
Joints:
- removed joint camera_joint
- added joint tube_joint: type fixed, parent vacuum_base_link, child vacuum_tcp, origin xyz=0 0.25 0 rpy=0 0 0
