Commit message: online execution working

File: rubyrhod_ws/src/doosan-robot/dsr_description/xacro/macro.m1013.white.xacro (robot description, xacro)
@@ -11,6 +11,6 @@
 				<origin xyz="-3.4e-05   -0.004815    0.048482"/>
 				<inertia ixx="0.016331" ixy="-6.4837e-06" ixz="2.0048e-06" iyy="0.014945"
-					iyz="-0.00051686"
-					izz="0.022577"/>
+						 iyz="-0.00051686"
+						 izz="0.022577"/>
 			</inertial>
 			<visual>
@@ -35,12 +35,12 @@
 				<origin xyz="0.000119      0.0428   -0.006383"/>
 				<inertia ixx="0.04506" ixy="4.1126e-05" ixz="-5.2533e-05" iyy="0.029679"
-					iyz="-0.0019959"
-					izz="0.047056"/>
-			</inertial>
-            <collision>
-                <geometry>
-                    <cylinder radius="0.1" length="0.2"/>
-                </geometry>
-            </collision>
+						 iyz="-0.0019959"
+						 izz="0.047056"/>
+			</inertial>
+			<collision>
+				<geometry>
+					<cylinder radius="0.1" length="0.2"/>
+				</geometry>
+			</collision>
 			<visual>
 				<origin rpy="0 0 0" xyz="0 0 0" />
@@ -64,13 +64,13 @@
 				<origin xyz="0.25973    -5.3e-05     0.15782"/>
 				<inertia ixx="0.037586" ixy="-0.00036999" ixz="-0.0069927" iyy="0.84943"
-					iyz="4.0201e-05"
-					izz="0.85021"/>
-			</inertial>
-            <collision>
-                <origin rpy="0 -1.571 0" xyz="0.3 0 0.1525" />
-                <geometry>
-                    <cylinder radius="0.08" length="0.75"/>
-                </geometry>
-            </collision>
+						 iyz="4.0201e-05"
+						 izz="0.85021"/>
+			</inertial>
+			<collision>
+				<origin rpy="0 -1.571 0" xyz="0.3 0 0.1525" />
+				<geometry>
+					<cylinder radius="0.08" length="0.75"/>
+				</geometry>
+			</collision>
 			<visual>
 				<origin rpy="0 0 0" xyz="0 0 0" />
@@ -106,8 +106,8 @@
 				<origin xyz="-1.5e-05   -0.006702    0.044608"/>
 				<inertia ixx="0.018748" ixy="7.8071e-06" ixz="-5.0324e-06" iyy="0.018972"
-					iyz="-0.00099342"
-					izz="0.011502"/>
-			</inertial>
-            <visual>
+						 iyz="-0.00099342"
+						 izz="0.011502"/>
+			</inertial>
+			<visual>
 				<origin rpy="0 0 0" xyz="0 0 0" />
 				<geometry>
@@ -130,12 +130,12 @@
 				<origin xyz="7.1e-05    0.091879    -0.18252"/>
 				<inertia ixx="0.19063" ixy="-1.8037e-05" ixz="-3.8576e-05" iyy="0.17268" iyz="-0.052996"
-					izz="0.030386"/>
-			</inertial>
-            <collision>
-                <origin rpy="-0.55 0 0" xyz="0 0.07 -0.3" />
-                <geometry>
-                    <cylinder radius="0.07" length="0.4"/>
-                </geometry>
-            </collision>
+						 izz="0.030386"/>
+			</inertial>
+			<collision>
+				<origin rpy="-0.55 0 0" xyz="0 0.07 -0.3" />
+				<geometry>
+					<cylinder radius="0.07" length="0.4"/>
+				</geometry>
+			</collision>
 			<visual>
 				<origin rpy="0 0 0" xyz="0 0 0" />
@@ -165,19 +165,19 @@
 				<origin xyz="-0.000273    0.003651    0.032088"/>
 				<inertia ixx="0.015583" ixy="2.135e-05" ixz="-5.1895e-06" iyy="0.011519"
-					iyz="0.00042553"
-					izz="0.0088671"/>
-			</inertial>
-            <collision>
-                <origin rpy="1.571 0 0" xyz="0 0 0" />
-                <geometry>
-                    <cylinder radius="0.08" length="0.15"/>
-                </geometry>
-            </collision>
-			<collision>
-                <origin rpy="0 0 0" xyz="0 0 0.15" />
-                <geometry>
-                    <cylinder radius="0.08" length="0.15"/>
-                </geometry>
-            </collision>
+						 iyz="0.00042553"
+						 izz="0.0088671"/>
+			</inertial>
+			<collision>
+				<origin rpy="1.571 0 0" xyz="0 0 0" />
+				<geometry>
+					<cylinder radius="0.08" length="0.15"/>
+				</geometry>
+			</collision>
+			<collision>
+				<origin rpy="0 0 0" xyz="0 0 0.15" />
+				<geometry>
+					<cylinder radius="0.08" length="0.15"/>
+				</geometry>
+			</collision>
 			<visual>
 				<origin rpy="0 0 0" xyz="0 0 0" />
@@ -201,6 +201,6 @@
 				<origin xyz="-0.000292       7e-06     -0.0539"/>
 				<inertia ixx="0.0048282" ixy="4.1298e-06" ixz="6.9879e-06" iyy="0.0059519"
-					iyz="4.252e-06"
-					izz="0.0061263"/>
+						 iyz="4.252e-06"
+						 izz="0.0061263"/>
 			</inertial>
 			<visual>

File: rubyrhod_ws/src/doosan-robot/moveit_config_m1013/config/gazebo_m1013.urdf (robot description, URDF)
Before this commit: robot m1013, 14 links, 13 joints
Links:
- added link vacuum_safe_tcp
- added link vacuum_sphere, mass 0.1; collision sphere radius=0.024; visual sphere radius=0.024
- added link vacuum_tube, mass 0.1; collision cylinder length=0.128 radius=0.012; visual cylinder length=0.128 radius=0.012
- link vacuum_base_link: geometry collision mesh filename=package://vacuum/meshes/tool.STL scale=0.0010 0.0010 0.0010; visual mesh filename=package://vacuum/meshes/tool.STL scale=0.001 0.001 0.001
- link vacuum_tcp: mass 0.1 -> None; geometry 
Joints:
- added joint sphere_joint: type fixed, parent vacuum_tube, child vacuum_sphere, origin xyz=0 0.128 0 rpy=0 0 0
- added joint tcp_joint: type fixed, parent vacuum_sphere, child vacuum_tcp, origin xyz=0 0.048 0 rpy=0 0 0
- added joint tcp_safe_joint: type fixed, parent vacuum_tcp, child vacuum_safe_tcp, origin xyz=0 0.05 0 rpy=0 0 0
- joint joint1: limit lower=-6.2832 upper=6.2832 effort=346 velocity=2.0944 -> lower=-1.5708 upper=0.785398 effort=346 velocity=2.0944
- joint joint4: limit lower=-6.2832 upper=6.2832 effort=50 velocity=3.927 -> lower=0 upper=6.2832 effort=50 velocity=3.927
- joint joint5: limit lower=-6.2832 upper=6.2832 effort=50 velocity=3.927 -> lower=-1.74533 upper=1.57 effort=50 velocity=3.927
- joint joint6: limit lower=-6.2832 upper=6.2832 effort=50 velocity=3.927 -> lower=-3.1415 upper=0 effort=50 velocity=3.927
- joint tube_joint: child vacuum_tcp -> vacuum_tube; origin xyz=0 0.25 0 rpy=0 0 0 -> xyz=0 0.1 0 rpy=0 0 0

File: rubyrhod_ws/src/vacuum/urdf/vacuum.urdf (robot description, URDF)
Before this commit: robot vacuum, 4 links, 3 joints
Links:
- added link vacuum_sphere; collision sphere radius=0.024; visual sphere radius=0.024
- link vacuum_tube: geometry collision cylinder length=0.128 radius=0.012; visual cylinder length=0.128 radius=0.012
Joints:
- added joint sphere_joint: type fixed, parent vacuum_tube, child vacuum_sphere, origin xyz=0 0.128 0 rpy=0 0 0
- joint tcp_joint: origin xyz=0 0.15 0 rpy=0 0 0 -> xyz=0 0.048 0 rpy=0 0 0; parent vacuum_tube -> vacuum_sphere
- joint tube_joint: origin xyz=0 0.105 0 rpy=0 0 0 -> xyz=0 0.1 0 rpy=0 0 0
