Commit message: End of test

File: rubyrhod_ws/src/doosan-robot/dsr_description/xacro/m1013.urdf.xacro (robot description, xacro)
@@ -38,8 +38,19 @@
   <xacro:include filename="$(find azure_kinect_ros_driver)/urdf/azure_kinect.urdf.xacro" />
   <joint name="camera_fixed" type="fixed">
-    <origin xyz="-0.05 0 0.1" rpy="0 -1.57 0"/>
+    <origin xyz="-0.06 0.01 0.1" rpy="-1.15622991 -1.56390655  1.14494029"/>
     <parent link="link6"/>
     <child link="camera_base"/>
   </joint>
+<!--  Matrice entre link6 et camera_base -->
+<!--  0.00582503  0.00730799   -0.999956  -0.0744662-->
+<!--  0.00419196    0.999964  0.00733246  0.00341612-->
+<!--  0.999974 -0.00423448  0.00579419    0.102301-->
+<!--  0           0           0           1-->
+<!--  0.0028461   0.0112804   -0.999932  -0.0737303-->
+<!--  0.00627436    0.999916   0.0112981 0.000351512-->
+<!--  0.999976 -0.00630609  0.00277508    0.102236-->
+<!--  0           0           0           1-->
+<!--  Angle XYZ -->
+<!-- x:-0.9020437, y: -1.5614485, z: -0.8978304 -->
   <xacro:include filename="$(find vacuum)/urdf/vacuum.urdf"/>
   <joint name="vacuum_fixed" type="fixed">

File: rubyrhod_ws/src/doosan-robot/dsr_description/xacro/macro.m1013.white.xacro (robot description, xacro)
@@ -27,5 +27,5 @@
 			<origin rpy="0 0 0" xyz="0 0 0.1525" />
 			<axis xyz="0 0 1" />
-			<limit effort="346" lower="-3.1415" upper="1.57" velocity="2.0944"/>
+			<limit effort="346" lower="-1.5708" upper="1.5708" velocity="2.0944"/>
 			<dynamics friction="0" />
 		</joint>
@@ -157,5 +157,5 @@
 			<origin rpy="-1.571 0 0" xyz="0 0 0" />
 			<axis xyz="0 0 1" />
-			<limit effort="50" lower="-1.57" upper="1.57" velocity="3.927"/>
+			<limit effort="50" lower="-1.58825" upper="1.91986" velocity="3.927"/>
 			<dynamics friction="0" />
 		</joint>

File: rubyrhod_ws/src/doosan-robot/moveit_config_m1013/config/gazebo_m1013.urdf (robot description, URDF)
Before this commit: robot m1013, 17 links, 16 joints
Links:
- link camera_base: geometry collision box size=0.039 0.1545 0.0585; visual box size=0.026 0.103 0.039
- link camera_body: geometry collision box size=0.1491 0.1494 0.0345; visual box size=0.0994 0.0996 0.023
- link camera_visor: geometry collision box size=0.039 0.1515 0.0555; visual box size=0.026 0.101 0.037
- link vacuum_base_link: geometry collision box size=0.18 0.15 0.15; visual mesh filename=package://vacuum/meshes/tool.STL scale=0.001 0.001 0.001
- link vacuum_sphere: geometry collision sphere radius=0.020; visual sphere radius=0.015
Joints:
- joint camera_fixed: origin xyz=-0.05 0 0.1 rpy=0 -1.57 0 -> xyz=-0.08 -0.01 0.1 rpy=0 -1.57 0
- joint joint1: limit lower=-1.5708 upper=0.785398 effort=346 velocity=2.0944 -> lower=-1.5708 upper=1.5708 effort=346 velocity=2.0944
- joint joint2: limit lower=-6.2832 upper=6.2832 effort=346 velocity=2.0944 -> lower=-3.1415 upper=3.1415 effort=346 velocity=2.0944
- joint joint4: limit lower=0 upper=6.2832 effort=50 velocity=3.927 -> lower=-3.1415 upper=3.1415 effort=50 velocity=3.927
- joint joint5: limit lower=-1.74533 upper=1.57 effort=50 velocity=3.927 -> lower=-1.58825 upper=1.91986 effort=50 velocity=3.927
- joint joint6: limit lower=-3.1415 upper=0 effort=50 velocity=3.927 -> lower=-2.61799 upper=0.872665 effort=50 velocity=3.927
- joint tube_joint: origin xyz=0 0.1 0 rpy=0 0 0 -> xyz=0 0.13 0 rpy=0 0 0
