Commit message: online wotking during 15-20 min

File: rubyrhod_ws/src/Azure_Kinect_ROS_Driver/urdf/azure_kinect.urdf.xacro (robot description, xacro)
@@ -28,5 +28,5 @@
     <collision>
       <geometry>
-          <box size="0.0994 0.0996 0.023" />
+          <box size="0.1491 0.1494 0.0345" />
       </geometry>
     </collision>
@@ -42,5 +42,5 @@
     <collision>
       <geometry>
-          <box size="0.026 0.103 0.039" />
+          <box size="0.039 0.1545 0.0585" />
       </geometry>
     </collision>
@@ -56,5 +56,5 @@
     <collision>
       <geometry>
-          <box size="0.026 0.101 0.037" />
+          <box size="0.039 0.1515 0.0555" />
       </geometry>
     </collision>

File: rubyrhod_ws/src/doosan-robot/dsr_description/xacro/macro.m1013.white.xacro (robot description, xacro)
@@ -27,5 +27,5 @@
 			<origin rpy="0 0 0" xyz="0 0 0.1525" />
 			<axis xyz="0 0 1" />
-			<limit effort="346" lower="-1.5708" upper="0.785398" velocity="2.0944"/>
+			<limit effort="346" lower="-3.1415" upper="1.57" velocity="2.0944"/>
 			<dynamics friction="0" />
 		</joint>
@@ -56,5 +56,5 @@
 			<origin rpy="0 -1.571 -1.571" xyz="0 0.0345 0" />
 			<axis xyz="0 0 1" />
-			<limit effort="346" lower="-6.2832" upper="6.2832" velocity="2.0944"/>
+			<limit effort="346" lower="-3.1415" upper="3.1415" velocity="2.0944"/>
 			<dynamics friction="0" />
 		</joint>
@@ -122,5 +122,5 @@
 			<origin rpy="1.571 0 0" xyz="0 -0.559 0" />
 			<axis xyz="0 0 1" />
-			<limit effort="50" lower="0" upper="6.2832" velocity="3.927"/>
+			<limit effort="50" lower="-3.1415" upper="3.1415" velocity="3.927"/>
 			<dynamics friction="0" />
 		</joint>
@@ -157,5 +157,5 @@
 			<origin rpy="-1.571 0 0" xyz="0 0 0" />
 			<axis xyz="0 0 1" />
-			<limit effort="50" lower="-1.74533" upper="1.57" velocity="3.927"/>
+			<limit effort="50" lower="-1.57" upper="1.57" velocity="3.927"/>
 			<dynamics friction="0" />
 		</joint>
@@ -193,5 +193,5 @@
 			<origin rpy="1.571 0 0" xyz="0 -0.121 0" />
 			<axis xyz="0 0 1" />
-			<limit effort="50" lower="-3.1415" upper="0" velocity="3.927"/>
+			<limit effort="50" lower="-2.61799" upper="0.872665" velocity="3.927"/>
 			<dynamics friction="0" />
 		</joint>

File: rubyrhod_ws/src/vacuum/urdf/vacuum.urdf (robot description, URDF)
Before this commit: robot vacuum, 5 links, 4 joints
Links:
- link vacuum_base_link: geometry collision box size=0.18 0.15 0.15; visual mesh filename=package://vacuum/meshes/tool.STL scale=0.001 0.001 0.001
