Commit message: End of test

File: rubyrhod_ws/src/vacuum/urdf/vacuum.urdf (robot description, URDF)
Before this commit: robot vacuum, 5 links, 4 joints
Links:
- link vacuum_sphere: geometry collision sphere radius=0.020; visual sphere radius=0.015
Joints:
- joint tube_joint: origin xyz=0 0.1 0 rpy=0 0 0 -> xyz=0 0.13 0 rpy=0 0 0
